File: Board/ARDEC-controller-v1.brd (EAGLE design)
At the start: 55.9 x 95.2 mm, 27 parts, among them IC1 L293D, IC2 L293D, IC4 MEGA8-P, IC5 7805T, Q2 16MHz

Commit message: Version 2.0
Connections:
- removed net IO3: BUTTONS.5, IC4.5
- new net N$15: IC2.7, IC4.5
- net IO10/SS: now also BUTTONS.5; no longer IC1.7
- net IO13/SCK: now also IC1.7; no longer IC2.7
Routing:
- net N$15: track 0.00 -> 42.5 mm, vias 0 -> 1
- net IO10/SS: track 24.4 -> 56.6 mm, vias 1 -> 2
- net IO3: track 13.8 -> 0.00 mm
- net IO13/SCK: track 74.4 -> 81.4 mm
